File: kitchen_lights.sch (KiCad schematic (older format))
At the start: 66 parts, among them IC1 ATTINY24/44/84-SSU, IC2 MBI5168, P1 CONN_6, P2 CONN_6, P3 CONN_1, P4 CONN_1, P5 CONN_1, P6 CONN_1, P7 CONN_1, P8 CONN_1, Q1 CSTLA_T, SW1 LPH_SW, SW2 LPH_SW, SW3 LPH_SW, U1 7805MS

Commit message: Upgrades... added a small prototyping area for the remaining pins.
Parts:
- removed Q1: CSTLA_T, murata-resonators-CSTLA_T, symbol CSTLA_T
- added P10, P9: CONN_1, symbol CONN_1
- added P11, P12, P13, P14: CONN_6, symbol CONN_6
- renumbered U1 to IC3
Connections:
- net labels added: LED, PA0, PA2, PA3, PA7
- net labels removed: RESERVED, XTAL1, XTAL2
- wire segments 164 -> 172
- no-connect marks 9 -> 26
Other:
- moved on the sheet: D33, P3, P4, P5, P6, P7, P8, R10

Commit message: Reworked the board, now calling it 'V1.01'.
Parts:
- removed P1, P11, P2: CONN_6, symbol CONN_6
- added C7, C8: 2.2mF, symbol CP1
- added P1, P2: CONN_8, symbol CONN_8
- RV1: value POT -> I_REF
- renumbered P3 to MH0, P4 to MH1, P5 to MH2, P6 to MH3, P7 to MH4, P8 to MH5, P9 to MH6, P10 to MH7, P12 to P4, P13 to P5, P14 to P6
Connections:
- net GND: now also P4.2, P5.2
- net GNDPWR: now also C7.2, C8.2, P1.7 (P7), P1.8 (P8), P2.7 (P7), P2.8 (P8)
- net PA0: now also P1.1 (P1), P2.1 (P1)
- net PA2: now also P4.5, P5.5, P6.2, P1.3 (P3), P2.3 (P3); no longer P6.1
- net PA3: now also P4.4, P5.4, P6.3, P1.4 (P4), P2.4 (P4); no longer P6.2
- net RESET: now also P4.3, P5.3
- net SWITCHES: now also IC1.6 ((PCINT7/ICP/OC0B/ADC7)PA7); no longer IC1.12 ((PCINT1/AIN0/ADC1)PA1)
- net VCC: now also P4.1, P5.1
- net V_LED: now also C7.1, C8.1, P1.5 (P5), P1.6 (P6), P2.5 (P5), P2.6 (P6)
- net PA1: now reaches P4.6
- net PA1: now also IC1.12 ((PCINT1/AIN0/ADC1)PA1), P5.6, P6.1, P1.2 (P2), P2.2 (P2)
- removed net PA7: IC1.6 ((PCINT7/ICP/OC0B/ADC7)PA7), P6.3
- no-connect marks 26 -> 8
Other:
- moved on the sheet: P4, P5, P6
